Commit message: Tuned

File: smb_description/urdf/smb_properties.urdf.xacro (robot description, xacro)
@@ -11,5 +11,5 @@
     <xacro:property name="topMass" value="0.001"/>
     <xacro:property name="wheelWidth" value="0.08"/>
-    <xacro:property name="wheelRadius" value="0.14"/>
+    <xacro:property name="wheelRadius" value="0.195"/>
     <xacro:property name="frontWheelX" value="0.2159"/>
     <xacro:property name="backWheelX" value="-0.2159"/>
