Commit message: fix frictionless wheel and remove unused components of smb xacro file

File: smb_description/urdf/smb.urdf.xacro (robot description, xacro)
@@ -1,18 +1,27 @@
 <?xml version="1.0"?>
 <robot xmlns:xacro="http://www.ros.org/wiki/xacro" name="smb">
+    <!-- TODO: replace this arg by other ones like sensors, legacy, etc -->
     <xacro:arg name="lidar" default="true"/>
+    <!-- Defines colors and calculates typical inertias -->
     <xacro:include filename="$(find smb_description)/urdf/smb_utils.urdf.xacro" />
+    <!-- Defines IMU macro -->
     <xacro:include filename="$(find smb_description)/urdf/sensor_plugins/smb_imu.gazebo.xacro"/>
+    <!-- Defines GPS macro -->
     <xacro:include filename="$(find smb_description)/urdf/sensor_plugins/smb_gps.gazebo.xacro"/>
     <xacro:if value="$(arg lidar)">
         <xacro:include filename="$(find smb_description)/urdf/sensor_plugins/smb_robosense.gazebo.xacro"/>
     </xacro:if>
+    <!-- Defines odometry macro -->
     <xacro:include filename="$(find smb_description)/urdf/sensor_plugins/smb_odometry.gazebo.xacro"/>
+    <!-- Defines lidar macro -->
     <xacro:include filename="$(find smb_description)/urdf/realsense_t265.urdf.xacro"/>
+    <!-- Defines camera macro -->
     <xacro:include filename="$(find smb_description)/urdf/sensor_plugins/smb_mono.gazebo.xacro"/>
+    <!-- Defines blackfly camera macro -->
     <xacro:include filename="$(find smb_description)/urdf/smb_blackfly_camera.urdf.xacro"/>
+    <!-- Defines blackfly stereo macro -->
     <xacro:include filename="$(find smb_description)/urdf/smb_blackfly_camera_stereo.urdf.xacro"/>
+    <!-- Defines lidar macro -->
     <xacro:include filename="$(find smb_description)/urdf/smb_lidar_mount.urdf.xacro"/>
-    <xacro:property name="PI" value="3.1415926535897931"/>
     <!-- Model macros -->
     <xacro:macro name="wheel" params="prefix X Y wheel_joint_type friction_coeff:=0.2 transmission_reduction:=${wheelTransmission}" >
@@ -146,6 +155,5 @@
         <xacro:wheel prefix="LH" X="${backWheelX}"
             Y="${chassisWidth/2+wheelClearance+wheelWidth/2}"
-	    wheel_joint_type="${wheel_joint_type}"
-        friction_coeff="0.0" />
+	    wheel_joint_type="${wheel_joint_type}" />
         <xacro:wheel prefix="RH" X="${backWheelX}"
             Y="${-chassisWidth/2-wheelClearance-wheelWidth/2}"
@@ -153,5 +161,5 @@
         <xacro:IMU base_link="${base_link_name}" simulation="${simulation}"/>
         <!-- <xacro:GPS base_link="${base_link_name}" simulation="${simulation}"/> -->
-        <xacro:mono_cam base_link="${base_link_name}" simulation="${simulation}"/>
+        <!-- <xacro:mono_cam base_link="${base_link_name}" simulation="${simulation}"/>
         <xacro:blackfly_cam id="0" base_link="${base_link_name}" simulation="${simulation}">
             <origin xyz="0.29082 0.04458 ${0.0955 + chassisHeight/2.0}" rpy="0 0 0" />
@@ -160,5 +168,5 @@
             <origin xyz="0.29082 -0.04542 ${0.0955 + chassisHeight/2.0}" rpy="0 0 0" />
         </xacro:blackfly_cam>
-        <xacro:blackfly_cam_stereo base_link="${base_link_name}" simulation="${simulation}"/>
+        <xacro:blackfly_cam_stereo base_link="${base_link_name}" simulation="${simulation}"/> -->
         <xacro:if value="${lidar}">
             <xacro:LIDAR base_link="${base_link_name}" simulation="${simulation}"/>

File: smb_description/urdf/smb_standalone.urdf.xacro (robot description, xacro)
@@ -13,8 +13,9 @@
   <xacro:property name="lidar" value="$(arg lidar)"/>
   <!-- Includes -->
+  <!-- This loads a bunch of xacro properties -->
   <xacro:include filename="$(find smb_description)/urdf/smb_big_properties.urdf.xacro" />
-  <xacro:if value="$(arg simulation)">
+  <!-- <xacro:if value="$(arg simulation)">
     <xacro:include filename="$(find smb_description)/urdf/smb_gazebo_addins.urdf.xacro"/>
-  </xacro:if>
+  </xacro:if> -->
   <xacro:include filename="$(find smb_description)/urdf/smb.urdf.xacro">
     <xacro:arg name="lidar" default="$(arg lidar)"/>

Commit message: Improve Gazebo simulation (#21)
* Change configuration files: add back wheels and reduce max velocity and accelleration

* Set ekf to false since we are using only the tracking camera

* fix frictionless wheel and remove unused components of smb xacro file

* added missing component back

* Fix friction coefficients for gazebo simulation

* Fix typo

* Remove joint from left and right wheel parameter

Co-authored-by: David Oort Alonso <davidoort@hotmail.com>

File: smb_description/urdf/smb.urdf.xacro (robot description, xacro)
@@ -1,18 +1,27 @@
 <?xml version="1.0"?>
 <robot xmlns:xacro="http://www.ros.org/wiki/xacro" name="smb">
+    <!-- TODO: replace this arg by other ones like sensors, legacy, etc -->
     <xacro:arg name="lidar" default="true"/>
+    <!-- Defines colors and calculates typical inertias -->
     <xacro:include filename="$(find smb_description)/urdf/smb_utils.urdf.xacro" />
+    <!-- Defines IMU macro -->
     <xacro:include filename="$(find smb_description)/urdf/sensor_plugins/smb_imu.gazebo.xacro"/>
+    <!-- Defines GPS macro -->
     <xacro:include filename="$(find smb_description)/urdf/sensor_plugins/smb_gps.gazebo.xacro"/>
     <xacro:if value="$(arg lidar)">
         <xacro:include filename="$(find smb_description)/urdf/sensor_plugins/smb_robosense.gazebo.xacro"/>
     </xacro:if>
+    <!-- Defines odometry macro -->
     <xacro:include filename="$(find smb_description)/urdf/sensor_plugins/smb_odometry.gazebo.xacro"/>
+    <!-- Defines lidar macro -->
     <xacro:include filename="$(find smb_description)/urdf/realsense_t265.urdf.xacro"/>
+    <!-- Defines camera macro -->
     <xacro:include filename="$(find smb_description)/urdf/sensor_plugins/smb_mono.gazebo.xacro"/>
+    <!-- Defines blackfly camera macro -->
     <xacro:include filename="$(find smb_description)/urdf/smb_blackfly_camera.urdf.xacro"/>
+    <!-- Defines blackfly stereo macro -->
     <xacro:include filename="$(find smb_description)/urdf/smb_blackfly_camera_stereo.urdf.xacro"/>
+    <!-- Defines lidar macro -->
     <xacro:include filename="$(find smb_description)/urdf/smb_lidar_mount.urdf.xacro"/>
-    <xacro:property name="PI" value="3.1415926535897931"/>
     <!-- Model macros -->
     <xacro:macro name="wheel" params="prefix X Y wheel_joint_type friction_coeff:=0.2 transmission_reduction:=${wheelTransmission}" >
@@ -139,19 +148,20 @@
             Y="${chassisWidth/2+wheelClearance+wheelWidth/2}"
             wheel_joint_type="${wheel_joint_type}"
-            friction_coeff="0.5" />
+            friction_coeff="0.7" />
         <xacro:wheel prefix="RF" X="${frontWheelX}"
             Y="${-chassisWidth/2-wheelClearance-wheelWidth/2}"
             wheel_joint_type="${wheel_joint_type}"
-            friction_coeff="0.5"/>
+            friction_coeff="0.7"/>
         <xacro:wheel prefix="LH" X="${backWheelX}"
             Y="${chassisWidth/2+wheelClearance+wheelWidth/2}"
-	    wheel_joint_type="${wheel_joint_type}"
-        friction_coeff="0.0" />
+	        wheel_joint_type="${wheel_joint_type}"
+            friction_coeff="0.7"/>
         <xacro:wheel prefix="RH" X="${backWheelX}"
             Y="${-chassisWidth/2-wheelClearance-wheelWidth/2}"
-            wheel_joint_type="${wheel_joint_type}" />
+            wheel_joint_type="${wheel_joint_type}"
+            friction_coeff="0.7"/>
         <xacro:IMU base_link="${base_link_name}" simulation="${simulation}"/>
         <!-- <xacro:GPS base_link="${base_link_name}" simulation="${simulation}"/> -->
-        <xacro:mono_cam base_link="${base_link_name}" simulation="${simulation}"/>
+        <!-- <xacro:mono_cam base_link="${base_link_name}" simulation="${simulation}"/>
         <xacro:blackfly_cam id="0" base_link="${base_link_name}" simulation="${simulation}">
             <origin xyz="0.29082 0.04458 ${0.0955 + chassisHeight/2.0}" rpy="0 0 0" />
@@ -160,5 +170,5 @@
             <origin xyz="0.29082 -0.04542 ${0.0955 + chassisHeight/2.0}" rpy="0 0 0" />
         </xacro:blackfly_cam>
-        <xacro:blackfly_cam_stereo base_link="${base_link_name}" simulation="${simulation}"/>
+        <xacro:blackfly_cam_stereo base_link="${base_link_name}" simulation="${simulation}"/> -->
         <xacro:if value="${lidar}">
             <xacro:LIDAR base_link="${base_link_name}" simulation="${simulation}"/>

Commit message: Put mono camera back into smb urdf

File: smb_description/urdf/smb.urdf.xacro (robot description, xacro)
@@ -163,10 +163,11 @@
         <xacro:IMU base_link="${base_link_name}" simulation="${simulation}"/>
         <!-- <xacro:GPS base_link="${base_link_name}" simulation="${simulation}"/> -->
-        <!-- <xacro:mono_cam base_link="${base_link_name}" simulation="${simulation}"/>
-        <xacro:blackfly_cam id="0" base_link="${base_link_name}" simulation="${simulation}">
+        <!-- <xacro:mono_cam base_link="${base_link_name}" simulation="${simulation}"/> -->
+        <xacro:blackfly_cam id="_right" base_link="${base_link_name}" simulation="${simulation}">
+            <origin xyz="0.29082 -0.04542 ${0.0955 + chassisHeight/2.0}" rpy="0 0 0" />
+        </xacro:blackfly_cam>
+        <!--
+        <xacro:blackfly_cam id="_left" base_link="${base_link_name}" simulation="${simulation}">
             <origin xyz="0.29082 0.04458 ${0.0955 + chassisHeight/2.0}" rpy="0 0 0" />
-        </xacro:blackfly_cam>
-        <xacro:blackfly_cam id="1" base_link="${base_link_name}" simulation="${simulation}">
-            <origin xyz="0.29082 -0.04542 ${0.0955 + chassisHeight/2.0}" rpy="0 0 0" />
         </xacro:blackfly_cam>
         <xacro:blackfly_cam_stereo base_link="${base_link_name}" simulation="${simulation}"/> -->

Commit message: WIP: Disabling tracking camera by default
Properly exposing argument to control tracking camera (enabled/disabled) . Setting default to disabled.

File: smb_description/urdf/smb.urdf.xacro (robot description, xacro)
@@ -3,4 +3,5 @@
     <!-- TODO: replace this arg by other ones like sensors, legacy, etc -->
     <xacro:arg name="lidar" default="true"/>
+    <xacro:arg name="tracking_camera" default="false"/>
     <!-- Defines colors and calculates typical inertias -->
     <xacro:include filename="$(find smb_description)/urdf/smb_utils.urdf.xacro" />
@@ -14,5 +15,7 @@
     <xacro:include filename="$(find smb_description)/urdf/sensor_plugins/smb_odometry.gazebo.xacro"/>
     <!-- Defines realsense_t265 (tracking camera) macro -->
-    <xacro:include filename="$(find smb_description)/urdf/realsense_t265.urdf.xacro"/>
+    <xacro:if value="$(arg tracking_camera)">
+        <xacro:include filename="$(find smb_description)/urdf/realsense_t265.urdf.xacro"/>
+    </xacro:if>
     <!-- Defines blackfly rgbcamera camera macro -->
     <xacro:include filename="$(find smb_description)/urdf/smb_rgbcamera.urdf.xacro"/>
@@ -24,5 +27,5 @@
             <parent link="${base_link_name}"/>
             <child link="${prefix}_WHEEL"/>
-            <origin xyz="${X} ${Y} ${wheelHeight - chassisHeight/2.0}" rpy="-${0.5*PI} 0 0" />
+            <origin xyz="${X} ${Y} ${wheelHeight - chassisHeight/2.0}" rpy="-${0.5*M_PI} 0 0" />
             <axis xyz="0 0 1" rpy="0 0 0" />
             <dynamics damping="1.0" friction="0.0"/>
@@ -138,5 +141,5 @@
     </link>
     </xacro:macro>
-    <xacro:macro name="smb" params="wheel_joint_type:=continuous lidar:=${lidar} tracking_camera:=true simulation:=true">
+    <xacro:macro name="smb" params="wheel_joint_type:=continuous lidar:=$(arg lidar) tracking_camera:=$(arg tracking_camera) simulation:=true">
         <xacro:chassis/>
         <xacro:wheel prefix="LF" X="${frontWheelX}"

File: smb_description/urdf/smb_standalone.urdf.xacro (robot description, xacro)
@@ -9,5 +9,5 @@
   <xacro:arg name="description_name_xacro"    default="robot_description"/>
   <xacro:arg name="publish_tf"                default="false"/>
-  <xacro:arg name="tracking_camera"           default="true"/>
+  <xacro:arg name="tracking_camera"           default="false"/>
   <xacro:property name="lidar" value="$(arg lidar)"/>
   <!-- Includes -->
@@ -17,7 +17,5 @@
     <xacro:include filename="$(find smb_description)/urdf/smb_gazebo_addins.urdf.xacro"/>
   </xacro:if>
-  <xacro:include filename="$(find smb_description)/urdf/smb.urdf.xacro">
-    <xacro:arg name="lidar" default="$(arg lidar)"/>
-  </xacro:include>
+  <xacro:include filename="$(find smb_description)/urdf/smb.urdf.xacro" />
   <xacro:smb wheel_joint_type="$(arg wheel_joint_type)" simulation="$(arg simulation)" tracking_camera="$(arg tracking_camera)"/>
 </robot>
