Commit message: merge branch dev/slam_toolbox

File: smb_description/urdf/realsense_t265.urdf.xacro (robot description, xacro)
@@ -56,8 +56,8 @@
       <origin xyz="0 ${realsense_t265_housing_center_x_offset} 0 " rpy="${0.5*PI} 0 ${-0.5*PI}" />
     </joint>
-    <link name="realsense_t265_imu_optical_frame" />
+    <link name="camera_imu_optical_frame" />
     <joint name="realsense_t265_imu_joint" type="fixed">
       <parent link="realsense_t265_odom_frame"/>
-      <child link="realsense_t265_imu_optical_frame"/>
+      <child link="camera_imu_optical_frame"/>
       <origin xyz="0 0 0 " rpy="0 ${PI} 0" />
     </joint>

File: smb_description/urdf/sensor_plugins/smb_imu.gazebo.xacro (robot description, xacro)
@@ -79,4 +79,16 @@
       </material>
     </link>
+    <link name="imu">
+      <inertial>
+        <mass value="0.001"/>
+        <origin rpy="0 0 0" xyz="0 0 0"/>
+        <inertia ixx="0.0001" ixy="0" ixz="0" iyy="0.000001" iyz="0" izz="0.0001"/>
+      </inertial>
+    </link>
+    <joint name="imu_imu_link_joint" type="fixed">
+      <origin xyz="0 0 0" rpy="0 0 0"/>
+      <parent link="${imu_link}"/>
+      <child link="imu"/>
+    </joint>
     <gazebo reference="${imu_link}">
       <material>Gazebo/Orange</material>

Commit message: A lot of cleanup of urdf model - Deleting obsolete files - Renaming macros for more consistency - adjusting topic names

File: smb_description/urdf/realsense_t265.urdf.xacro (robot description, xacro)
@@ -14,5 +14,5 @@
        https://www.intel.com/content/dam/support/us/en/documents/emerging-technologies/intel-realsense-technology/IntelRealSenseTrackingT265Datasheet.pdf -->
   <xacro:macro name="REALSENSE_T265" params="base_link t265_origin_xyz t265_origin_rpy simulation">
-    <link name="realsense_t265">
+    <link name="tracking_camera_link">
       <inertial>
           <mass value="0.001"/>
@@ -34,38 +34,39 @@
       </visual>
     </link>
-    <gazebo reference="realsense_t265">
+    <gazebo reference="tracking_camera_link">
         <material>Gazebo/Black</material>
     </gazebo>
-    <joint name="realsense_t265_joint" type="fixed">
+    <joint name="tracking_camera_joint" type="fixed">
       <parent link="${base_link}"/>
-      <child link="realsense_t265"/>
-      <!-- <origin xyz="-${chassisLength/2.0+realsense_t265_width} 0.0 ${chassisHeight*0.5+realsense_t265_height*0.5}" rpy="0 0 ${PI}" /> -->
+      <child link="tracking_camera_link"/>
       <!-- Manually calibrated sensor orientation  -->
       <origin xyz="${t265_origin_xyz}" rpy="${t265_origin_rpy}" />
     </joint>
-    <joint name="camera_pose_frame_joint" type="fixed">
-      <parent link="realsense_t265"/>
-      <child link="camera_pose_frame"/>
+    <gazebo reference="tracking_camera_joint">
+      <disableFixedJointLumping>true</disableFixedJointLumping>
+    </gazebo>
+    <link name="tracking_camera_pose_frame" />
+    <joint name="tracking_camera_pose_frame_joint" type="fixed">
+      <parent link="tracking_camera_link"/>
+      <child link="tracking_camera_pose_frame"/>
       <origin xyz="0 0 0" rpy="0 0 0" />
     </joint>
-    <link name="camera_pose_frame" />
-    <link name="realsense_t265_odom_frame" />
-    <joint name="realsense_t265_odom_joint" type="fixed">
-      <parent link="realsense_t265"/>
-      <child link="realsense_t265_odom_frame"/>
+    <link name="tracking_camera_odom_frame" />
+    <joint name="tracking_camera_odom_joint" type="fixed">
+      <parent link="tracking_camera_link"/>
+      <child link="tracking_camera_odom_frame"/>
       <origin xyz="0 ${realsense_t265_housing_center_x_offset} 0 " rpy="${0.5*PI} 0 ${-0.5*PI}" />
     </joint>
-    <link name="camera_imu_optical_frame" />
-    <joint name="realsense_t265_imu_joint" type="fixed">
-      <parent link="realsense_t265_odom_frame"/>
-      <child link="camera_imu_optical_frame"/>
+    <!--
+    <link name="tracking_camera_optical_frame" />
+    <joint name="tracking_camera_optical_joint" type="fixed">
+      <parent link="tracking_camera_odom_frame"/>
+      <child link="tracking_camera_optical_frame"/>
       <origin xyz="0 0 0 " rpy="0 ${PI} 0" />
     </joint>
-      <xacro:if value="${simulation}">
-            <xacro:odometry_plugin sensor_link="realsense_t265" topic_name="/tracking_camera/odom/sample" rate="200" max_linear_speed_before_settle="0.01" max_angular_speed_before_settle="0.05" publish_tf="false"/>
-      </xacro:if>
-      <gazebo reference="realsense_t265_joint">
-          <disableFixedJointLumping>true</disableFixedJointLumping>
-      </gazebo>
+    -->
+    <xacro:if value="${simulation}">
+          <xacro:odometry_plugin sensor_link="tracking_camera_link" topic_name="/tracking_camera/odom/sample" odom_frame="tracking_camera_odom_frame" child_odom_frame="tracking_camera_pose_frame" rate="200" max_linear_speed_before_settle="0.01" max_angular_speed_before_settle="0.05" publish_tf="false"/>
+    </xacro:if>
   </xacro:macro>
 </robot>

File: smb_description/urdf/sensor_plugins/smb_rgbcamera.gazebo.xacro (robot description, xacro)
@@ -1,9 +1,9 @@
 <?xml version="1.0"?>
 <robot name="smb" xmlns:xacro="http://www.ros.org/wiki/xacro">
-  <xacro:macro name="rgbcamera_camera_plugin" params="name rate">
-    <xacro:property name="camera_topic" value="/visual_inertial_sensor/cam0/slow/image_raw" />
-    <xacro:property name="camera_info_topic" value="/visual_inertial_sensor/cam0/slow/camera_info" />
-    <gazebo reference="${name}_link">
-      <sensor type="camera" name="${name}_cam">
+  <xacro:macro name="rgbcamera_camera_plugin" params="name link_name rate">
+    <xacro:property name="camera_topic" value="/${name}/image_raw" />
+    <xacro:property name="camera_info_topic" value="/${name}/camera_info" />
+    <gazebo reference="${link_name}">
+      <sensor type="camera" name="${name}">
         <pose>0.0066 0 0 0 0 0</pose>
         <visualize>false</visualize>
@@ -22,8 +22,4 @@
           <noise>
             <type>gaussian</type>
-            <!-- Noise parameters based on published spec for Hokuyo laser
-                achieving "+-30mm" accuracy at range < 10m.  A mean of 0.0m and
-                stddev of 0.01m will put 99.7% of samples within 0.03m of the true
-                reading. -->
             <mean>0.0</mean>
             <stddev>0.007</stddev>
@@ -33,5 +29,5 @@
           <alwaysOn>true</alwaysOn>
           <updateRate>0.0</updateRate>
-          <cameraName>${name}_cam</cameraName>
+          <cameraName>${name}</cameraName>
           <imageTopicName>${camera_topic}</imageTopicName>
           <cameraInfoTopicName>${camera_info_topic}</cameraInfoTopicName>

File: smb_description/urdf/sensor_plugins/smb_robosense.gazebo.xacro (robot description, xacro)
@@ -5,9 +5,9 @@
   <xacro:arg name="pointcloud_topic"	default="/rslidar/points"/>
   <xacro:property name="gpu" 		value="$(arg gpu)" />
-  <xacro:macro name="LIDAR" params="base_link simulation">
+  <xacro:macro name="LIDAR" params="parent_link simulation">
     <xacro:if value="${simulation}">
       <xacro:include filename="$(find robosense_description)/urdf/RS-16.urdf.xacro"/>
-      <xacro:RS-16 parent="${base_link}" name="rslidar" topic="$(arg pointcloud_topic)" hz="10" samples="440" gpu="${gpu}">
-        <origin xyz="0.0245 0 ${payloadHeight+lidarBoxHeight+chassisHeight/2.0}" rpy="0 0 0" />
+      <xacro:RS-16 parent="${parent_link}" name="rslidar" topic="$(arg pointcloud_topic)" hz="10" samples="440" gpu="${gpu}">
+        <origin xyz="0.0 0.0 ${lidarBoxHeight}" rpy="0 0 0" />
       </xacro:RS-16>
       <gazebo reference="rslidar_base_mount_joint">
@@ -18,6 +18,8 @@
       </gazebo>
       <!--  simulate icp-->
+      <!--
       <xacro:include filename="$(find smb_description)/urdf/sensor_plugins/smb_odometry.gazebo.xacro"/>
       <xacro:odometry_plugin sensor_link="rslidar" topic_name="/rslidar/ground_truth" odom_frame="map" child_odom_frame="lidar" publish_tf="false"/>
+      -->
     </xacro:if>
     <xacro:unless value="${simulation}">
@@ -38,8 +40,8 @@
           </visual>
       </link>
-      <joint name="base_to_rslidar" type="fixed">
-        <parent link="${base_link}"/>
+      <joint name="${parent_link}_to_rslidar" type="fixed">
+        <parent link="${parent_link}"/>
         <child link="rslidar"/>
-        <origin xyz="0.0245 0 ${payloadHeight+lidarBoxHeight+chassisHeight/2.0+0.038}" rpy="0 0 0"/>
+        <origin xyz="0.0 0.0 ${lidarBoxHeight+0.039}" rpy="0 0 0"/>
       </joint>
     </xacro:unless>

File: smb_description/urdf/smb.urdf.xacro (robot description, xacro)
@@ -7,6 +7,5 @@
     <!-- Defines IMU macro -->
     <xacro:include filename="$(find smb_description)/urdf/sensor_plugins/smb_imu.gazebo.xacro"/>
-    <!-- Defines GPS macro -->
-    <xacro:include filename="$(find smb_description)/urdf/sensor_plugins/smb_gps.gazebo.xacro"/>
+    <!-- Defines Lidar macro -->
     <xacro:if value="$(arg lidar)">
         <xacro:include filename="$(find smb_description)/urdf/sensor_plugins/smb_robosense.gazebo.xacro"/>
@@ -14,12 +13,8 @@
     <!-- Defines odometry macro -->
     <xacro:include filename="$(find smb_description)/urdf/sensor_plugins/smb_odometry.gazebo.xacro"/>
-    <!-- Defines lidar macro -->
+    <!-- Defines realsense_t265 (tracking camera) macro -->
     <xacro:include filename="$(find smb_description)/urdf/realsense_t265.urdf.xacro"/>
-    <!-- Defines camera macro -->
-    <xacro:include filename="$(find smb_description)/urdf/sensor_plugins/smb_mono.gazebo.xacro"/>
-    <!-- Defines blackfly camera macro -->
-    <xacro:include filename="$(find smb_description)/urdf/smb_blackfly_camera.urdf.xacro"/>
-    <!-- Defines blackfly stereo macro -->
-    <xacro:include filename="$(find smb_description)/urdf/smb_blackfly_camera_stereo.urdf.xacro"/>
+    <!-- Defines blackfly rgbcamera camera macro -->
+    <xacro:include filename="$(find smb_description)/urdf/smb_rgbcamera.urdf.xacro"/>
     <!-- Defines lidar macro -->
     <xacro:include filename="$(find smb_description)/urdf/smb_lidar_mount.urdf.xacro"/>
@@ -143,5 +138,5 @@
     </link>
     </xacro:macro>
-    <xacro:macro name="smb" params="wheel_joint_type:=continuous lidar:=${lidar} tracking_camera:=true tracking_camera_rear_facing:=false simulation:=true">
+    <xacro:macro name="smb" params="wheel_joint_type:=continuous lidar:=${lidar} tracking_camera:=true simulation:=true">
         <xacro:chassis/>
         <xacro:wheel prefix="LF" X="${frontWheelX}"
@@ -163,30 +158,16 @@
         <xacro:IMU base_link="${base_link_name}" simulation="${simulation}"/>
         <!-- <xacro:GPS base_link="${base_link_name}" simulation="${simulation}"/> -->
-        <!-- <xacro:mono_cam base_link="${base_link_name}" simulation="${simulation}"/> -->
-        <xacro:rgbcamera_cam id="_right" base_link="${base_link_name}" simulation="${simulation}">
+        <xacro:rgbcamera_cam id="" base_link="${base_link_name}" simulation="${simulation}">
             <origin xyz="0.29082 -0.04542 ${0.0955 + chassisHeight/2.0}" rpy="0 0 0" />
         </xacro:rgbcamera_cam>
-        <!--
-        <xacro:rgbcamera_cam id="_left" base_link="${base_link_name}" simulation="${simulation}">
-            <origin xyz="0.29082 0.04458 ${0.0955 + chassisHeight/2.0}" rpy="0 0 0" />
-        </xacro:rgbcamera_cam>
-        <xacro:rgbcamera_cam_stereo base_link="${base_link_name}" simulation="${simulation}"/> -->
         <xacro:if value="${lidar}">
-            <xacro:LIDAR base_link="${base_link_name}" simulation="${simulation}"/>
             <xacro:lidar_mount base_link="${base_link_name}"/>
+            <xacro:LIDAR parent_link="lidar_mount_link" simulation="${simulation}"/>
         </xacro:if>
         <xacro:if value="${tracking_camera}">
-            <xacro:unless value="${tracking_camera_rear_facing}">
-                <xacro:REALSENSE_T265 base_link="imu_link"
-                    t265_origin_xyz="0.0537 0.0321 0.172"
-                    t265_origin_rpy="0 0 0"
-                    simulation="${simulation}"/>
-            </xacro:unless>
-            <xacro:if value="${tracking_camera_rear_facing}">
-                <xacro:REALSENSE_T265 base_link="imu_link"
-                    t265_origin_xyz="${0.0537-0.6} 0.0321 0.172"
-                    t265_origin_rpy="0 0 ${PI}"
-                    simulation="${simulation}"/>
-            </xacro:if>
+            <xacro:REALSENSE_T265 base_link="base_link"
+                t265_origin_xyz="0.309 0.008 0.352"
+                t265_origin_rpy="0 0 0"
+                simulation="${simulation}"/>
         </xacro:if>
     </xacro:macro>

File: smb_description/urdf/smb_gazebo_addins.urdf.xacro (robot description, xacro)
@@ -1,11 +1,5 @@
 <?xml version="1.0"?>
 <robot xmlns:xacro="http://www.ros.org/wiki/xacro" name="smb">
-  <xacro:arg name="use_ros_skid_steer" default="false"/>
   <xacro:arg name="use_ros_control" default="false"/>
-  <xacro:if value="$(arg use_ros_skid_steer)">
-    <xacro:include filename="$(find smb_description)/urdf/smb_ros_skid_steer.gazebo.xacro"/>
-    <xacro:smb_ros_skid_steer_plugin description_name="$(arg description_name_xacro)"
-      broadcast_tf="true" robot_namespace="$(arg robot_namespace)"/>
-  </xacro:if>
   <xacro:if value="$(arg use_ros_control)">
     <xacro:include filename="$(find smb_description)/urdf/smb_ros_control.gazebo.xacro"/>

File: smb_description/urdf/smb_lidar_mount.urdf.xacro (robot description, xacro)
@@ -28,7 +28,4 @@
       <child link="lidar_mount_link"/>
     </joint>
-    <gazebo reference="lidar_mount_joint">
-      <disableFixedJointLumping>true</disableFixedJointLumping>
-    </gazebo>
   </xacro:macro>
 </robot>

File: smb_description/urdf/smb_rgbcamera.urdf.xacro (robot description, xacro)
@@ -4,5 +4,5 @@
 <robot name="smb" xmlns:xacro="http://www.ros.org/wiki/xacro">
   <!-- INCLUDE PLUGIN -->
-  <xacro:include filename="$(find smb_description)/urdf/sensor_plugins/smb_blackfly.gazebo.xacro"/>
+  <xacro:include filename="$(find smb_description)/urdf/sensor_plugins/smb_rgbcamera.gazebo.xacro"/>
   <xacro:macro name="rgbcamera_cam" params="*origin id base_link simulation">
     <!--                              Camera  Properties 				          	-->
@@ -50,5 +50,5 @@
     </joint>
     <xacro:if value="${simulation}">
-        <xacro:rgbcamera_camera_plugin name="rgbcamera${id}" rate="${rgbcamera_update_rate}"/>
+        <xacro:rgbcamera_camera_plugin name="rgb_camera" link_name="${rgbcamera_link}" rate="${rgbcamera_update_rate}"/>
     </xacro:if>
   </xacro:macro>

File: smb_description/urdf/smb_standalone.urdf.xacro (robot description, xacro)
@@ -4,5 +4,4 @@
   <xacro:arg name="wheel_joint_type"          default="fixed"/> <!-- continuous for gazebo -->
   <xacro:arg name="simulation"                default="false"/>
-  <xacro:arg name="use_ros_skid_steer"        default="false"/> <!-- Specify one! -->
   <xacro:arg name="use_ros_control"           default="false"/>
   <xacro:arg name="lidar"                     default="true"/>
