Commit message: cleanup and renaming of topic names (#38)
* modified:   odometry_conversion/src/OdometryConversion.cpp
	modified:   record_sensors.sh
	modified:   smb/launch/smb.launch
	modified:   smb_description/urdf/realsense_t265.urdf.xacro
	modified:   smb_slam/config/localization/param_with_camera_odometry.yaml
	modified:   smb_slam/config/localization/param_with_lidar_odometry.yaml
	modified:   smb_slam/smb_tf_publisher.py

* versavis

* lidar+imu

* blackfly+mpc

* modified:   launch/sensors.launch
	modified:   launch/smb.launch
	modified:   package.xml

* Fixing bug in odometry conversion node

* A lot of cleanup of urdf model
- Deleting obsolete files
- Renaming macros for more consistency
- adjusting topic names

* Adding launch file to odometry_conversion

* Adapting OdometryConversion
switching transform direction of tf published by OdometryConversion
--> necessary such that base_link can be child of odom frame

* Cleaning up tracking cam frames

* Publishing tf of odometry_plugin in simulation
Instead of using the OdometryConversion node,
the odom tf is now published directly by the gazebo odometry plugin.

Why hasn't this been done before?

* Tested changes on real robot
Adjusted things to make it work on real robot
todo @mantelt: check sim again!

* Again use OdometryConversion also in sim

Instead of publishing the tf of the odometry_plugin,
use the OdometryConversion tool again to
publish odom tf of tracking camera (as on real robot).

* WIP: Disabling tracking camera by default

Properly exposing argument to control tracking camera (enabled/disabled) . Setting default to disabled.

* getting keyboard teleop and soft e stop in control namespace

---------

Co-authored-by: duandaxia <felicity.duan@gmail.com>
Co-authored-by: Shobhit Singhal <shobhitsinghal55@gmail.com>

File: smb_description/urdf/realsense_t265.urdf.xacro (robot description, xacro)
@@ -14,5 +14,5 @@
        https://www.intel.com/content/dam/support/us/en/documents/emerging-technologies/intel-realsense-technology/IntelRealSenseTrackingT265Datasheet.pdf -->
   <xacro:macro name="REALSENSE_T265" params="base_link t265_origin_xyz t265_origin_rpy simulation">
-    <link name="realsense_t265">
+    <link name="tracking_camera_link">
       <inertial>
           <mass value="0.001"/>
@@ -34,38 +34,41 @@
       </visual>
     </link>
-    <gazebo reference="realsense_t265">
+    <gazebo reference="tracking_camera_link">
         <material>Gazebo/Black</material>
     </gazebo>
-    <joint name="realsense_t265_joint" type="fixed">
+    <joint name="tracking_camera_joint" type="fixed">
       <parent link="${base_link}"/>
-      <child link="realsense_t265"/>
-      <!-- <origin xyz="-${chassisLength/2.0+realsense_t265_width} 0.0 ${chassisHeight*0.5+realsense_t265_height*0.5}" rpy="0 0 ${PI}" /> -->
+      <child link="tracking_camera_link"/>
       <!-- Manually calibrated sensor orientation  -->
       <origin xyz="${t265_origin_xyz}" rpy="${t265_origin_rpy}" />
     </joint>
-    <joint name="camera_pose_frame_joint" type="fixed">
-      <parent link="realsense_t265"/>
-      <child link="camera_pose_frame"/>
+    <gazebo reference="tracking_camera_joint">
+      <disableFixedJointLumping>true</disableFixedJointLumping>
+    </gazebo>
+    <link name="tracking_camera_pose_frame" />
+    <joint name="tracking_camera_pose_frame_joint" type="fixed">
+      <parent link="tracking_camera_link"/>
+      <child link="tracking_camera_pose_frame"/>
       <origin xyz="0 0 0" rpy="0 0 0" />
     </joint>
-    <link name="camera_pose_frame" />
-    <link name="realsense_t265_odom_frame" />
-    <joint name="realsense_t265_odom_joint" type="fixed">
-      <parent link="realsense_t265"/>
-      <child link="realsense_t265_odom_frame"/>
+    <!--
+    <link name="tracking_camera_odom_frame" />
+    <joint name="tracking_camera_odom_joint" type="fixed">
+      <parent link="tracking_camera_link"/>
+      <child link="tracking_camera_odom_frame"/>
       <origin xyz="0 ${realsense_t265_housing_center_x_offset} 0 " rpy="${0.5*PI} 0 ${-0.5*PI}" />
     </joint>
-    <link name="camera_imu_optical_frame" />
-    <joint name="realsense_t265_imu_joint" type="fixed">
-      <parent link="realsense_t265_odom_frame"/>
-      <child link="camera_imu_optical_frame"/>
+    -->
+    <!--
+    <link name="tracking_camera_optical_frame" />
+    <joint name="tracking_camera_optical_joint" type="fixed">
+      <parent link="tracking_camera_odom_frame"/>
+      <child link="tracking_camera_optical_frame"/>
       <origin xyz="0 0 0 " rpy="0 ${PI} 0" />
     </joint>
-      <xacro:if value="${simulation}">
-            <xacro:odometry_plugin sensor_link="realsense_t265" topic_name="/camera/odom/sample" rate="200" max_linear_speed_before_settle="0.01" max_angular_speed_before_settle="0.05" publish_tf="false"/>
-      </xacro:if>
-      <gazebo reference="realsense_t265_joint">
-          <disableFixedJointLumping>true</disableFixedJointLumping>
-      </gazebo>
+    -->
+    <xacro:if value="${simulation}">
+          <xacro:odometry_plugin sensor_link="tracking_camera_link" topic_name="/tracking_camera/odom/sample" odom_frame="tracking_camera_odom" rate="200" max_linear_speed_before_settle="0.01" max_angular_speed_before_settle="0.05" publish_tf="false"/>
+    </xacro:if>
   </xacro:macro>
 </robot>

File: smb_description/urdf/sensor_plugins/smb_rgbcamera.gazebo.xacro (robot description, xacro)
@@ -1,9 +1,9 @@
 <?xml version="1.0"?>
 <robot name="smb" xmlns:xacro="http://www.ros.org/wiki/xacro">
-  <xacro:macro name="blackfly_camera_plugin" params="name rate">
-    <xacro:property name="camera_topic" value="/versavis/cam0/slow/image_raw" />
-    <xacro:property name="camera_info_topic" value="/versavis/cam0/slow/camera_info" />
-    <gazebo reference="${name}_link">
-      <sensor type="camera" name="${name}_cam">
+  <xacro:macro name="rgbcamera_camera_plugin" params="name link_name rate">
+    <xacro:property name="camera_topic" value="/${name}/image_raw" />
+    <xacro:property name="camera_info_topic" value="/${name}/camera_info" />
+    <gazebo reference="${link_name}">
+      <sensor type="camera" name="${name}">
         <pose>0.0066 0 0 0 0 0</pose>
         <visualize>false</visualize>
@@ -22,8 +22,4 @@
           <noise>
             <type>gaussian</type>
-            <!-- Noise parameters based on published spec for Hokuyo laser
-                achieving "+-30mm" accuracy at range < 10m.  A mean of 0.0m and
-                stddev of 0.01m will put 99.7% of samples within 0.03m of the true
-                reading. -->
             <mean>0.0</mean>
             <stddev>0.007</stddev>
@@ -33,5 +29,5 @@
           <alwaysOn>true</alwaysOn>
           <updateRate>0.0</updateRate>
-          <cameraName>${name}_cam</cameraName>
+          <cameraName>${name}</cameraName>
           <imageTopicName>${camera_topic}</imageTopicName>
           <cameraInfoTopicName>${camera_info_topic}</cameraInfoTopicName>

File: smb_description/urdf/sensor_plugins/smb_robosense.gazebo.xacro (robot description, xacro)
@@ -3,11 +3,11 @@
   <xacro:arg name="simulation"   		default="false"/>
   <xacro:arg name="gpu" 		 		default="false"/>
-  <xacro:arg name="pointcloud_topic"	default="/rslidar_points"/>
+  <xacro:arg name="pointcloud_topic"	default="/rslidar/points"/>
   <xacro:property name="gpu" 		value="$(arg gpu)" />
-  <xacro:macro name="LIDAR" params="base_link simulation">
+  <xacro:macro name="LIDAR" params="parent_link simulation">
     <xacro:if value="${simulation}">
       <xacro:include filename="$(find robosense_description)/urdf/RS-16.urdf.xacro"/>
-      <xacro:RS-16 parent="${base_link}" name="rslidar" topic="$(arg pointcloud_topic)" hz="10" samples="440" gpu="${gpu}">
-        <origin xyz="0.0245 0 ${payloadHeight+lidarBoxHeight+chassisHeight/2.0}" rpy="0 0 0" />
+      <xacro:RS-16 parent="${parent_link}" name="rslidar" topic="$(arg pointcloud_topic)" hz="10" samples="440" gpu="${gpu}">
+        <origin xyz="0.0 0.0 ${lidarBoxHeight}" rpy="0 0 0" />
       </xacro:RS-16>
       <gazebo reference="rslidar_base_mount_joint">
@@ -18,6 +18,8 @@
       </gazebo>
       <!--  simulate icp-->
+      <!--
       <xacro:include filename="$(find smb_description)/urdf/sensor_plugins/smb_odometry.gazebo.xacro"/>
-      <xacro:odometry_plugin sensor_link="rslidar" topic_name="/rslidar_ground_truth" odom_frame="map" child_odom_frame="lidar" publish_tf="false"/>
+      <xacro:odometry_plugin sensor_link="rslidar" topic_name="/rslidar/ground_truth" odom_frame="map" child_odom_frame="lidar" publish_tf="false"/>
+      -->
     </xacro:if>
     <xacro:unless value="${simulation}">
@@ -38,8 +40,8 @@
           </visual>
       </link>
-      <joint name="base_to_rslidar" type="fixed">
-        <parent link="${base_link}"/>
+      <joint name="${parent_link}_to_rslidar" type="fixed">
+        <parent link="${parent_link}"/>
         <child link="rslidar"/>
-        <origin xyz="0.0245 0 ${payloadHeight+lidarBoxHeight+chassisHeight/2.0+0.038}" rpy="0 0 0"/>
+        <origin xyz="0.0 0.0 ${lidarBoxHeight+0.039}" rpy="0 0 0"/>
       </joint>
     </xacro:unless>

File: smb_description/urdf/smb.urdf.xacro (robot description, xacro)
@@ -3,10 +3,10 @@
     <!-- TODO: replace this arg by other ones like sensors, legacy, etc -->
     <xacro:arg name="lidar" default="true"/>
+    <xacro:arg name="tracking_camera" default="false"/>
     <!-- Defines colors and calculates typical inertias -->
     <xacro:include filename="$(find smb_description)/urdf/smb_utils.urdf.xacro" />
     <!-- Defines IMU macro -->
     <xacro:include filename="$(find smb_description)/urdf/sensor_plugins/smb_imu.gazebo.xacro"/>
-    <!-- Defines GPS macro -->
-    <xacro:include filename="$(find smb_description)/urdf/sensor_plugins/smb_gps.gazebo.xacro"/>
+    <!-- Defines Lidar macro -->
     <xacro:if value="$(arg lidar)">
         <xacro:include filename="$(find smb_description)/urdf/sensor_plugins/smb_robosense.gazebo.xacro"/>
@@ -14,12 +14,10 @@
     <!-- Defines odometry macro -->
     <xacro:include filename="$(find smb_description)/urdf/sensor_plugins/smb_odometry.gazebo.xacro"/>
-    <!-- Defines lidar macro -->
-    <xacro:include filename="$(find smb_description)/urdf/realsense_t265.urdf.xacro"/>
-    <!-- Defines camera macro -->
-    <xacro:include filename="$(find smb_description)/urdf/sensor_plugins/smb_mono.gazebo.xacro"/>
-    <!-- Defines blackfly camera macro -->
-    <xacro:include filename="$(find smb_description)/urdf/smb_blackfly_camera.urdf.xacro"/>
-    <!-- Defines blackfly stereo macro -->
-    <xacro:include filename="$(find smb_description)/urdf/smb_blackfly_camera_stereo.urdf.xacro"/>
+    <!-- Defines realsense_t265 (tracking camera) macro -->
+    <xacro:if value="$(arg tracking_camera)">
+        <xacro:include filename="$(find smb_description)/urdf/realsense_t265.urdf.xacro"/>
+    </xacro:if>
+    <!-- Defines blackfly rgbcamera camera macro -->
+    <xacro:include filename="$(find smb_description)/urdf/smb_rgbcamera.urdf.xacro"/>
     <!-- Defines lidar macro -->
     <xacro:include filename="$(find smb_description)/urdf/smb_lidar_mount.urdf.xacro"/>
@@ -29,5 +27,5 @@
             <parent link="${base_link_name}"/>
             <child link="${prefix}_WHEEL"/>
-            <origin xyz="${X} ${Y} ${wheelHeight - chassisHeight/2.0}" rpy="-${0.5*PI} 0 0" />
+            <origin xyz="${X} ${Y} ${wheelHeight - chassisHeight/2.0}" rpy="-${0.5*M_PI} 0 0" />
             <axis xyz="0 0 1" rpy="0 0 0" />
             <dynamics damping="1.0" friction="0.0"/>
@@ -143,5 +141,5 @@
     </link>
     </xacro:macro>
-    <xacro:macro name="smb" params="wheel_joint_type:=continuous lidar:=${lidar} tracking_camera:=true tracking_camera_rear_facing:=false simulation:=true">
+    <xacro:macro name="smb" params="wheel_joint_type:=continuous lidar:=$(arg lidar) tracking_camera:=$(arg tracking_camera) simulation:=true">
         <xacro:chassis/>
         <xacro:wheel prefix="LF" X="${frontWheelX}"
@@ -163,30 +161,16 @@
         <xacro:IMU base_link="${base_link_name}" simulation="${simulation}"/>
         <!-- <xacro:GPS base_link="${base_link_name}" simulation="${simulation}"/> -->
-        <!-- <xacro:mono_cam base_link="${base_link_name}" simulation="${simulation}"/> -->
-        <xacro:blackfly_cam id="_right" base_link="${base_link_name}" simulation="${simulation}">
+        <xacro:rgbcamera_cam id="" base_link="${base_link_name}" simulation="${simulation}">
             <origin xyz="0.29082 -0.04542 ${0.0955 + chassisHeight/2.0}" rpy="0 0 0" />
-        </xacro:blackfly_cam>
-        <!--
-        <xacro:blackfly_cam id="_left" base_link="${base_link_name}" simulation="${simulation}">
-            <origin xyz="0.29082 0.04458 ${0.0955 + chassisHeight/2.0}" rpy="0 0 0" />
-        </xacro:blackfly_cam>
-        <xacro:blackfly_cam_stereo base_link="${base_link_name}" simulation="${simulation}"/> -->
+        </xacro:rgbcamera_cam>
         <xacro:if value="${lidar}">
-            <xacro:LIDAR base_link="${base_link_name}" simulation="${simulation}"/>
             <xacro:lidar_mount base_link="${base_link_name}"/>
+            <xacro:LIDAR parent_link="lidar_mount_link" simulation="${simulation}"/>
         </xacro:if>
         <xacro:if value="${tracking_camera}">
-            <xacro:unless value="${tracking_camera_rear_facing}">
-                <xacro:REALSENSE_T265 base_link="imu_link"
-                    t265_origin_xyz="0.0537 0.0321 0.172"
-                    t265_origin_rpy="0 0 0"
-                    simulation="${simulation}"/>
-            </xacro:unless>
-            <xacro:if value="${tracking_camera_rear_facing}">
-                <xacro:REALSENSE_T265 base_link="imu_link"
-                    t265_origin_xyz="${0.0537-0.6} 0.0321 0.172"
-                    t265_origin_rpy="0 0 ${PI}"
-                    simulation="${simulation}"/>
-            </xacro:if>
+            <xacro:REALSENSE_T265 base_link="base_link"
+                t265_origin_xyz="0.309 0.008 0.352"
+                t265_origin_rpy="0 0 0"
+                simulation="${simulation}"/>
         </xacro:if>
     </xacro:macro>

File: smb_description/urdf/smb_rgbcamera.urdf.xacro (robot description, xacro)
@@ -4,13 +4,13 @@
 <robot name="smb" xmlns:xacro="http://www.ros.org/wiki/xacro">
   <!-- INCLUDE PLUGIN -->
-  <xacro:include filename="$(find smb_description)/urdf/sensor_plugins/smb_blackfly.gazebo.xacro"/>
-  <xacro:macro name="blackfly_cam" params="*origin id base_link simulation">
+  <xacro:include filename="$(find smb_description)/urdf/sensor_plugins/smb_rgbcamera.gazebo.xacro"/>
+  <xacro:macro name="rgbcamera_cam" params="*origin id base_link simulation">
     <!--                              Camera  Properties 				          	-->
-    <xacro:property name="blackfly_base_link"		value="${base_link}"/>
-    <xacro:property name="blackfly_origin_rpy"		value="0 0 0"/>
-    <xacro:property name="blackfly_origin_xyz"		value="0.29082 -0.04458 ${0.0955 + chassisHeight/2.0}"/>
-    <xacro:property name="blackfly_update_rate"		value="2"/>
-    <xacro:property name="blackfly_link"  			value="blackfly${id}_link"/>
-    <link name="${blackfly_link}">
+    <xacro:property name="rgbcamera_base_link"		value="${base_link}"/>
+    <xacro:property name="rgbcamera_origin_rpy"		value="0 0 0"/>
+    <xacro:property name="rgbcamera_origin_xyz"		value="0.29082 -0.04458 ${0.0955 + chassisHeight/2.0}"/>
+    <xacro:property name="rgbcamera_update_rate"		value="2"/>
+    <xacro:property name="rgbcamera_link"  			value="rgbcamera${id}_link"/>
+    <link name="${rgbcamera_link}">
       <inertial>
         <mass value="0.01" /> <!-- [kg] -->
@@ -31,24 +31,24 @@
         </material>
     </link>
-      <gazebo reference="${blackfly_link}">
+      <gazebo reference="${rgbcamera_link}">
         <material>Gazebo/Red</material>
       </gazebo>
-    <joint name="blackfly${id}_camera_joint" type="fixed">
-      <!-- <origin xyz="${blackfly_origin_xyz}" rpy="${blackfly_origin_rpy}"/> -->
+    <joint name="rgbcamera${id}_camera_joint" type="fixed">
+      <!-- <origin xyz="${rgbcamera_origin_xyz}" rpy="${rgbcamera_origin_rpy}"/> -->
       <xacro:insert_block name="origin"/>
-      <parent link="${blackfly_base_link}"/>
-      <child link="${blackfly_link}"/>
+      <parent link="${rgbcamera_base_link}"/>
+      <child link="${rgbcamera_link}"/>
     </joint>
-      <gazebo reference="blackfly${id}_camera_joint">
+      <gazebo reference="rgbcamera${id}_camera_joint">
         <disableFixedJointLumping>true</disableFixedJointLumping>
       </gazebo>
-    <link name="blackfly${id}_optical_link"/>
-    <joint name="blackfly${id}_camera_optical_joint" type="fixed">
+    <link name="rgbcamera${id}_optical_link"/>
+    <joint name="rgbcamera${id}_camera_optical_joint" type="fixed">
       <origin xyz="0.0066 0 0" rpy="-1.57 0 -1.57"/>
-      <parent link="${blackfly_link}"/>
-      <child link="blackfly${id}_optical_link"/>
+      <parent link="${rgbcamera_link}"/>
+      <child link="rgbcamera${id}_optical_link"/>
     </joint>
     <xacro:if value="${simulation}">
-        <xacro:blackfly_camera_plugin name="blackfly${id}" rate="${blackfly_update_rate}"/>
+        <xacro:rgbcamera_camera_plugin name="rgb_camera" link_name="${rgbcamera_link}" rate="${rgbcamera_update_rate}"/>
     </xacro:if>
   </xacro:macro>

File: smb_description/urdf/smb_standalone.urdf.xacro (robot description, xacro)
@@ -4,5 +4,4 @@
   <xacro:arg name="wheel_joint_type"          default="fixed"/> <!-- continuous for gazebo -->
   <xacro:arg name="simulation"                default="false"/>
-  <xacro:arg name="use_ros_skid_steer"        default="false"/> <!-- Specify one! -->
   <xacro:arg name="use_ros_control"           default="false"/>
   <xacro:arg name="lidar"                     default="true"/>
@@ -10,5 +9,5 @@
   <xacro:arg name="description_name_xacro"    default="robot_description"/>
   <xacro:arg name="publish_tf"                default="false"/>
-  <xacro:arg name="tracking_camera"           default="true"/>
+  <xacro:arg name="tracking_camera"           default="false"/>
   <xacro:property name="lidar" value="$(arg lidar)"/>
   <!-- Includes -->
@@ -18,7 +17,5 @@
     <xacro:include filename="$(find smb_description)/urdf/smb_gazebo_addins.urdf.xacro"/>
   </xacro:if>
-  <xacro:include filename="$(find smb_description)/urdf/smb.urdf.xacro">
-    <xacro:arg name="lidar" default="$(arg lidar)"/>
-  </xacro:include>
+  <xacro:include filename="$(find smb_description)/urdf/smb.urdf.xacro" />
   <xacro:smb wheel_joint_type="$(arg wheel_joint_type)" simulation="$(arg simulation)" tracking_camera="$(arg tracking_camera)"/>
 </robot>
