Commit message: lidar+imu

File: smb_description/urdf/sensor_plugins/smb_imu.gazebo.xacro (robot description, xacro)
@@ -11,5 +11,5 @@
     <xacro:property name="imu_update_rate"		value="400"/>
     <xacro:property name="imu_link"  			value="imu_link"/>
-    <xacro:property name="imu_topic" 			value="/imu0"/>
+    <xacro:property name="imu_topic" 			value="/imu"/>
     <xacro:property name="imu_calibration_service_name" value="/imu/calibrate"/>
     <xacro:property name="acceleration_offset"          value="0.0 0.0 0.0"/>

File: smb_description/urdf/sensor_plugins/smb_robosense.gazebo.xacro (robot description, xacro)
@@ -3,5 +3,5 @@
   <xacro:arg name="simulation"   		default="false"/>
   <xacro:arg name="gpu" 		 		default="false"/>
-  <xacro:arg name="pointcloud_topic"	default="/rslidar_points"/>
+  <xacro:arg name="pointcloud_topic"	default="/rslidar/points"/>
   <xacro:property name="gpu" 		value="$(arg gpu)" />
   <xacro:macro name="LIDAR" params="base_link simulation">
@@ -19,5 +19,5 @@
       <!--  simulate icp-->
       <xacro:include filename="$(find smb_description)/urdf/sensor_plugins/smb_odometry.gazebo.xacro"/>
-      <xacro:odometry_plugin sensor_link="rslidar" topic_name="/rslidar_ground_truth" odom_frame="map" child_odom_frame="lidar" publish_tf="false"/>
+      <xacro:odometry_plugin sensor_link="rslidar" topic_name="/rslidar/ground_truth" odom_frame="map" child_odom_frame="lidar" publish_tf="false"/>
     </xacro:if>
     <xacro:unless value="${simulation}">
