Commit message: versavis

File: smb_description/urdf/sensor_plugins/smb_blackfly.gazebo.xacro (robot description, xacro)
@@ -2,6 +2,6 @@
 <robot name="smb" xmlns:xacro="http://www.ros.org/wiki/xacro">
   <xacro:macro name="blackfly_camera_plugin" params="name rate">
-    <xacro:property name="camera_topic" value="/versavis/cam0/slow/image_raw" />
-    <xacro:property name="camera_info_topic" value="/versavis/cam0/slow/camera_info" />
+    <xacro:property name="camera_topic" value="/visual_inertial_sensor/cam0/slow/image_raw" />
+    <xacro:property name="camera_info_topic" value="/visual_inertial_sensor/cam0/slow/camera_info" />
     <gazebo reference="${name}_link">
       <sensor type="camera" name="${name}_cam">

Commit message: blackfly+mpc

File: smb_description/urdf/sensor_plugins/smb_blackfly.gazebo.xacro (robot description, xacro)
@@ -1,5 +1,5 @@
 <?xml version="1.0"?>
 <robot name="smb" xmlns:xacro="http://www.ros.org/wiki/xacro">
-  <xacro:macro name="blackfly_camera_plugin" params="name rate">
+  <xacro:macro name="rgbcamera_camera_plugin" params="name rate">
     <xacro:property name="camera_topic" value="/visual_inertial_sensor/cam0/slow/image_raw" />
     <xacro:property name="camera_info_topic" value="/visual_inertial_sensor/cam0/slow/camera_info" />

File: smb_description/urdf/sensor_plugins/smb_blackfly_stereo.gazebo.xacro (robot description, xacro)
@@ -1,5 +1,5 @@
 <?xml version="1.0"?>
 <robot name="smb" xmlns:xacro="http://www.ros.org/wiki/xacro">
-<xacro:macro name="blackfly_camera_stereo_plugin" params="name rate">
+<xacro:macro name="rgbcamera_camera_stereo_plugin" params="name rate">
 <gazebo reference="${name}_left_link">
       <sensor type="multicamera" name="${name}_stereo_cam">

File: smb_description/urdf/smb.urdf.xacro (robot description, xacro)
@@ -164,12 +164,12 @@
         <!-- <xacro:GPS base_link="${base_link_name}" simulation="${simulation}"/> -->
         <!-- <xacro:mono_cam base_link="${base_link_name}" simulation="${simulation}"/> -->
-        <xacro:blackfly_cam id="_right" base_link="${base_link_name}" simulation="${simulation}">
+        <xacro:rgbcamera_cam id="_right" base_link="${base_link_name}" simulation="${simulation}">
             <origin xyz="0.29082 -0.04542 ${0.0955 + chassisHeight/2.0}" rpy="0 0 0" />
-        </xacro:blackfly_cam>
+        </xacro:rgbcamera_cam>
         <!--
-        <xacro:blackfly_cam id="_left" base_link="${base_link_name}" simulation="${simulation}">
+        <xacro:rgbcamera_cam id="_left" base_link="${base_link_name}" simulation="${simulation}">
             <origin xyz="0.29082 0.04458 ${0.0955 + chassisHeight/2.0}" rpy="0 0 0" />
-        </xacro:blackfly_cam>
-        <xacro:blackfly_cam_stereo base_link="${base_link_name}" simulation="${simulation}"/> -->
+        </xacro:rgbcamera_cam>
+        <xacro:rgbcamera_cam_stereo base_link="${base_link_name}" simulation="${simulation}"/> -->
         <xacro:if value="${lidar}">
             <xacro:LIDAR base_link="${base_link_name}" simulation="${simulation}"/>

File: smb_description/urdf/smb_blackfly_camera.urdf.xacro (robot description, xacro)
@@ -5,12 +5,12 @@
   <!-- INCLUDE PLUGIN -->
   <xacro:include filename="$(find smb_description)/urdf/sensor_plugins/smb_blackfly.gazebo.xacro"/>
-  <xacro:macro name="blackfly_cam" params="*origin id base_link simulation">
+  <xacro:macro name="rgbcamera_cam" params="*origin id base_link simulation">
     <!--                              Camera  Properties 				          	-->
-    <xacro:property name="blackfly_base_link"		value="${base_link}"/>
-    <xacro:property name="blackfly_origin_rpy"		value="0 0 0"/>
-    <xacro:property name="blackfly_origin_xyz"		value="0.29082 -0.04458 ${0.0955 + chassisHeight/2.0}"/>
-    <xacro:property name="blackfly_update_rate"		value="2"/>
-    <xacro:property name="blackfly_link"  			value="blackfly${id}_link"/>
-    <link name="${blackfly_link}">
+    <xacro:property name="rgbcamera_base_link"		value="${base_link}"/>
+    <xacro:property name="rgbcamera_origin_rpy"		value="0 0 0"/>
+    <xacro:property name="rgbcamera_origin_xyz"		value="0.29082 -0.04458 ${0.0955 + chassisHeight/2.0}"/>
+    <xacro:property name="rgbcamera_update_rate"		value="2"/>
+    <xacro:property name="rgbcamera_link"  			value="rgbcamera${id}_link"/>
+    <link name="${rgbcamera_link}">
       <inertial>
         <mass value="0.01" /> <!-- [kg] -->
@@ -31,24 +31,24 @@
         </material>
     </link>
-      <gazebo reference="${blackfly_link}">
+      <gazebo reference="${rgbcamera_link}">
         <material>Gazebo/Red</material>
       </gazebo>
-    <joint name="blackfly${id}_camera_joint" type="fixed">
-      <!-- <origin xyz="${blackfly_origin_xyz}" rpy="${blackfly_origin_rpy}"/> -->
+    <joint name="rgbcamera${id}_camera_joint" type="fixed">
+      <!-- <origin xyz="${rgbcamera_origin_xyz}" rpy="${rgbcamera_origin_rpy}"/> -->
       <xacro:insert_block name="origin"/>
-      <parent link="${blackfly_base_link}"/>
-      <child link="${blackfly_link}"/>
+      <parent link="${rgbcamera_base_link}"/>
+      <child link="${rgbcamera_link}"/>
     </joint>
-      <gazebo reference="blackfly${id}_camera_joint">
+      <gazebo reference="rgbcamera${id}_camera_joint">
         <disableFixedJointLumping>true</disableFixedJointLumping>
       </gazebo>
-    <link name="blackfly${id}_optical_link"/>
-    <joint name="blackfly${id}_camera_optical_joint" type="fixed">
+    <link name="rgbcamera${id}_optical_link"/>
+    <joint name="rgbcamera${id}_camera_optical_joint" type="fixed">
       <origin xyz="0.0066 0 0" rpy="-1.57 0 -1.57"/>
-      <parent link="${blackfly_link}"/>
-      <child link="blackfly${id}_optical_link"/>
+      <parent link="${rgbcamera_link}"/>
+      <child link="rgbcamera${id}_optical_link"/>
     </joint>
     <xacro:if value="${simulation}">
-        <xacro:blackfly_camera_plugin name="blackfly${id}" rate="${blackfly_update_rate}"/>
+        <xacro:rgbcamera_camera_plugin name="rgbcamera${id}" rate="${rgbcamera_update_rate}"/>
     </xacro:if>
   </xacro:macro>

File: smb_description/urdf/smb_blackfly_camera_stereo.urdf.xacro (robot description, xacro)
@@ -5,17 +5,17 @@
   <!-- INCLUDE PLUGIN -->
   <xacro:include filename="$(find smb_description)/urdf/sensor_plugins/smb_blackfly_stereo.gazebo.xacro"/>
-  <xacro:macro name="blackfly_cam_stereo" params="base_link simulation">
+  <xacro:macro name="rgbcamera_cam_stereo" params="base_link simulation">
     <!--                              Camera  Properties 				          	-->
-    <xacro:property name="blackfly_base_link"		value="${base_link}"/>
-    <xacro:property name="blackfly_left_origin_rpy"		value="0 0 0"/>
-    <xacro:property name="blackfly_left_origin_xyz"		value="0.29082 0.04458 ${0.0955 + chassisHeight/2.0}"/>
-    <xacro:property name="blackfly_right_origin_rpy"		value="0 0 0"/>
-    <xacro:property name="blackfly_right_origin_xyz"		value="0.29082 -0.04542 ${0.0955 + chassisHeight/2.0}"/>
-    <xacro:property name="blackfly_update_rate"		value="30"/>
-    <xacro:property name="blackfly_left_link"  		value="blackfly_left_link"/>
-    <xacro:property name="blackfly_right_link"  	value="blackfly_right_link"/>
-    <xacro:property name="blackfly_left_topic" 		value="/blackfly/left/image_raw"/>
-    <xacro:property name="blackfly_right_topic" 	value="/blackfly/right/image_raw"/>
-    <link name="${blackfly_left_link}">
+    <xacro:property name="rgbcamera_base_link"		value="${base_link}"/>
+    <xacro:property name="rgbcamera_left_origin_rpy"		value="0 0 0"/>
+    <xacro:property name="rgbcamera_left_origin_xyz"		value="0.29082 0.04458 ${0.0955 + chassisHeight/2.0}"/>
+    <xacro:property name="rgbcamera_right_origin_rpy"		value="0 0 0"/>
+    <xacro:property name="rgbcamera_right_origin_xyz"		value="0.29082 -0.04542 ${0.0955 + chassisHeight/2.0}"/>
+    <xacro:property name="rgbcamera_update_rate"		value="30"/>
+    <xacro:property name="rgbcamera_left_link"  		value="rgbcamera_left_link"/>
+    <xacro:property name="rgbcamera_right_link"  	value="rgbcamera_right_link"/>
+    <xacro:property name="rgbcamera_left_topic" 		value="/rgbcamera/left/image_raw"/>
+    <xacro:property name="rgbcamera_right_topic" 	value="/rgbcamera/right/image_raw"/>
+    <link name="${rgbcamera_left_link}">
       <inertial>
         <mass value="0.01" /> <!-- [kg] -->
@@ -36,8 +36,8 @@
         </material>
     </link>
-      <gazebo reference="${blackfly_left_link}">
+      <gazebo reference="${rgbcamera_left_link}">
         <material>Gazebo/Red</material>
       </gazebo>
-    <link name="${blackfly_right_link}">
+    <link name="${rgbcamera_right_link}">
       <inertial>
         <mass value="0.01" /> <!-- [kg] -->
@@ -58,37 +58,37 @@
         </material>
     </link>
-    <gazebo reference="${blackfly_right_link}">
+    <gazebo reference="${rgbcamera_right_link}">
         <material>Gazebo/Red</material>
       </gazebo>
-    <joint name="blackfly_left_camera_joint" type="fixed">
-      <origin xyz="${blackfly_left_origin_xyz}" rpy="${blackfly_left_origin_rpy}"/>
-      <parent link="${blackfly_base_link}"/>
-      <child link="${blackfly_left_link}"/>
+    <joint name="rgbcamera_left_camera_joint" type="fixed">
+      <origin xyz="${rgbcamera_left_origin_xyz}" rpy="${rgbcamera_left_origin_rpy}"/>
+      <parent link="${rgbcamera_base_link}"/>
+      <child link="${rgbcamera_left_link}"/>
     </joint>
-      <gazebo reference="blackfly_left_camera_joint">
+      <gazebo reference="rgbcamera_left_camera_joint">
         <disableFixedJointLumping>true</disableFixedJointLumping>
       </gazebo>
-    <joint name="blackfly_right_camera_joint" type="fixed">
-      <origin xyz="${blackfly_right_origin_xyz}" rpy="${blackfly_right_origin_rpy}"/>
-      <parent link="${blackfly_base_link}"/>
-      <child link="${blackfly_right_link}"/>
+    <joint name="rgbcamera_right_camera_joint" type="fixed">
+      <origin xyz="${rgbcamera_right_origin_xyz}" rpy="${rgbcamera_right_origin_rpy}"/>
+      <parent link="${rgbcamera_base_link}"/>
+      <child link="${rgbcamera_right_link}"/>
     </joint>
-      <gazebo reference="blackfly_right_camera_joint">
+      <gazebo reference="rgbcamera_right_camera_joint">
         <disableFixedJointLumping>true</disableFixedJointLumping>
       </gazebo>
-    <link name="blackfly_left_optical_link"/>
-    <link name="blackfly_right_optical_link"/>
-    <joint name="blackfly_left_camera_optical_joint" type="fixed">
+    <link name="rgbcamera_left_optical_link"/>
+    <link name="rgbcamera_right_optical_link"/>
+    <joint name="rgbcamera_left_camera_optical_joint" type="fixed">
       <origin xyz="0.0066 0 0" rpy="-1.57 0 -1.57"/>
-      <parent link="${blackfly_left_link}"/>
-      <child link="blackfly_left_optical_link"/>
+      <parent link="${rgbcamera_left_link}"/>
+      <child link="rgbcamera_left_optical_link"/>
     </joint>
-    <joint name="blackfly_right_camera_optical_joint" type="fixed">
+    <joint name="rgbcamera_right_camera_optical_joint" type="fixed">
       <origin xyz="0.0066 0 0" rpy="-1.57 0 -1.57"/>
-      <parent link="${blackfly_right_link}"/>
-      <child link="blackfly_right_optical_link"/>
+      <parent link="${rgbcamera_right_link}"/>
+      <child link="rgbcamera_right_optical_link"/>
     </joint>
     <xacro:if value="${simulation}">
-        <xacro:blackfly_camera_stereo_plugin name="blackfly" rate="${blackfly_update_rate}"/>
+        <xacro:rgbcamera_camera_stereo_plugin name="rgbcamera" rate="${rgbcamera_update_rate}"/>
     </xacro:if>
   </xacro:macro>
