Commit message: Add changes for lidar mount Add dae and stl files for mount Modify urdf files with correct transformations fix TF for open3d slam

File: smb_description/urdf/sensor_plugins/smb_robosense.gazebo.xacro (robot description, xacro)
@@ -9,5 +9,5 @@
       <xacro:include filename="$(find robosense_description)/urdf/RS-16.urdf.xacro"/>
       <xacro:RS-16 parent="${base_link}" name="rslidar" topic="$(arg pointcloud_topic)" hz="10" samples="440" gpu="${gpu}">
-        <origin xyz="0.00445 0 ${0.298+chassisHeight/2.0}" rpy="0 0 ${M_PI/2.0}" />
+        <origin xyz="0.0245 0 ${0.228+0.1+chassisHeight/2.0}" rpy="0 0 0" />
       </xacro:RS-16>
       <gazebo reference="rslidar_base_mount_joint">
@@ -41,5 +41,5 @@
         <parent link="${base_link}"/>
         <child link="rslidar"/>
-        <origin xyz="0.00445 0 ${0.298+chassisHeight/2.0+0.038}" rpy="0 0 ${M_PI/2.0}"/>
+        <origin xyz="0.0245 0 ${0.228+0.1+chassisHeight/2.0+0.038}" rpy="0 0 0"/>
       </joint>
     </xacro:unless>

File: smb_description/urdf/smb_lidar_mount.urdf.xacro (robot description, xacro)
@@ -7,9 +7,10 @@
     <xacro:property name="mount_base_link"		value="${base_link}"/>
     <xacro:property name="mount_origin_rpy"		value="0 0 0"/>
-    <xacro:property name="mount_origin_xyz"		value="0.00445 0 ${0.228+chassisHeight/2.0}"/>
+    <!-- <xacro:property name="mount_origin_xyz"		value="0.00445 0 ${0.228+chassisHeight/2.0}"/> -->
+    <xacro:property name="mount_origin_xyz"		value="0.0245 0 ${0.228+chassisHeight/2.0}"/>
     <link name="lidar_mount_link">
       <visual>
         <geometry>
-          <mesh filename="package://smb_description/urdf/new_payload/meshes/SMB_lidar_mount.dae"/>
+          <mesh filename="package://smb_description/urdf/new_payload/meshes/LidarBoxV2.dae"/>
         </geometry>
       </visual>

Commit message: Add params for xacro, cleanup

File: smb_description/urdf/sensor_plugins/smb_robosense.gazebo.xacro (robot description, xacro)
@@ -9,5 +9,5 @@
       <xacro:include filename="$(find robosense_description)/urdf/RS-16.urdf.xacro"/>
       <xacro:RS-16 parent="${base_link}" name="rslidar" topic="$(arg pointcloud_topic)" hz="10" samples="440" gpu="${gpu}">
-        <origin xyz="0.0245 0 ${0.228+0.1+chassisHeight/2.0}" rpy="0 0 0" />
+        <origin xyz="0.0245 0 ${payloadHeight+lidarBoxHeight+chassisHeight/2.0}" rpy="0 0 0" />
       </xacro:RS-16>
       <gazebo reference="rslidar_base_mount_joint">
@@ -41,5 +41,5 @@
         <parent link="${base_link}"/>
         <child link="rslidar"/>
-        <origin xyz="0.0245 0 ${0.228+0.1+chassisHeight/2.0+0.038}" rpy="0 0 0"/>
+        <origin xyz="0.0245 0 ${payloadHeight+lidarBoxHeight+chassisHeight/2.0+0.038}" rpy="0 0 0"/>
       </joint>
     </xacro:unless>

File: smb_description/urdf/smb_big_properties.urdf.xacro (robot description, xacro)
@@ -7,4 +7,6 @@
     <xacro:property name="chassisMass" value="40"/>
     <xacro:property name="M_PI"          value="3.14159265358"/>
+    <xacro:property name="payloadHeight" value="0.228"/>
+    <xacro:property name="lidarBoxHeight" value="0.1"/>
     <xacro:property name="topXOffset" value="-0.070"/>
     <xacro:property name="topHeight" value="0.180"/>

File: smb_description/urdf/smb_lidar_mount.urdf.xacro (robot description, xacro)
@@ -7,6 +7,5 @@
     <xacro:property name="mount_base_link"		value="${base_link}"/>
     <xacro:property name="mount_origin_rpy"		value="0 0 0"/>
-    <!-- <xacro:property name="mount_origin_xyz"		value="0.00445 0 ${0.228+chassisHeight/2.0}"/> -->
-    <xacro:property name="mount_origin_xyz"		value="0.0245 0 ${0.228+chassisHeight/2.0}"/>
+    <xacro:property name="mount_origin_xyz"		value="0.0245 0 ${payloadHeight+chassisHeight/2.0}"/>
     <link name="lidar_mount_link">
       <visual>

Commit message: New Lidar Mount and Open3d SLAM  (#36)
* Add localization mode for open3d slam

Add launch and param files for open3d slam localization
Add lua param files in smb slam from open3d slam
Modify mapping launch files

* Save modifications

* Add pcd map path

* Update Readme 

Running Instructions for Open3DSLAM

* Update README.md

* Update README.md

* Add changes for lidar mount
Add dae and stl files for mount
Modify urdf files with correct transformations
fix TF for open3d slam

* cleanup

remove icp localization
remove slam box
remove pointcloud stitcher
cleanup cmakelist
remove unnecessary launch files
remove tf publihser

* Add params for xacro, cleanup

* cleanup smb_slam

* Update README.md

* fix map save path

* cleanup cmake, package.xml in smb_slam

* Add launch files comment

* minor comments

File: smb_description/urdf/sensor_plugins/smb_robosense.gazebo.xacro (robot description, xacro)
@@ -9,5 +9,5 @@
       <xacro:include filename="$(find robosense_description)/urdf/RS-16.urdf.xacro"/>
       <xacro:RS-16 parent="${base_link}" name="rslidar" topic="$(arg pointcloud_topic)" hz="10" samples="440" gpu="${gpu}">
-        <origin xyz="0.00445 0 ${0.298+chassisHeight/2.0}" rpy="0 0 ${M_PI/2.0}" />
+        <origin xyz="0.0245 0 ${payloadHeight+lidarBoxHeight+chassisHeight/2.0}" rpy="0 0 0" />
       </xacro:RS-16>
       <gazebo reference="rslidar_base_mount_joint">
@@ -41,5 +41,5 @@
         <parent link="${base_link}"/>
         <child link="rslidar"/>
-        <origin xyz="0.00445 0 ${0.298+chassisHeight/2.0+0.038}" rpy="0 0 ${M_PI/2.0}"/>
+        <origin xyz="0.0245 0 ${payloadHeight+lidarBoxHeight+chassisHeight/2.0+0.038}" rpy="0 0 0"/>
       </joint>
     </xacro:unless>

File: smb_description/urdf/smb_lidar_mount.urdf.xacro (robot description, xacro)
@@ -7,9 +7,9 @@
     <xacro:property name="mount_base_link"		value="${base_link}"/>
     <xacro:property name="mount_origin_rpy"		value="0 0 0"/>
-    <xacro:property name="mount_origin_xyz"		value="0.00445 0 ${0.228+chassisHeight/2.0}"/>
+    <xacro:property name="mount_origin_xyz"		value="0.0245 0 ${payloadHeight+chassisHeight/2.0}"/>
     <link name="lidar_mount_link">
       <visual>
         <geometry>
-          <mesh filename="package://smb_description/urdf/new_payload/meshes/SMB_lidar_mount.dae"/>
+          <mesh filename="package://smb_description/urdf/new_payload/meshes/LidarBoxV2.dae"/>
         </geometry>
       </visual>
