Commit message: rgbcamera --> rgb_camera

File: smb_description/urdf/sensor_plugins/smb_rgb_camera.gazebo.xacro (robot description, xacro)
@@ -1,5 +1,5 @@
 <?xml version="1.0"?>
 <robot name="smb" xmlns:xacro="http://www.ros.org/wiki/xacro">
-  <xacro:macro name="rgbcamera_camera_plugin" params="name link_name rate">
+  <xacro:macro name="rgb_camera_camera_plugin" params="name link_name rate">
     <xacro:property name="camera_topic" value="/${name}/image_raw" />
     <xacro:property name="camera_info_topic" value="/${name}/camera_info" />

File: smb_description/urdf/smb.urdf.xacro (robot description, xacro)
@@ -18,6 +18,6 @@
         <xacro:include filename="$(find smb_description)/urdf/realsense_t265.urdf.xacro"/>
     </xacro:if>
-    <!-- Defines blackfly rgbcamera camera macro -->
-    <xacro:include filename="$(find smb_description)/urdf/smb_rgbcamera.urdf.xacro"/>
+    <!-- Defines blackfly rgb_camera camera macro -->
+    <xacro:include filename="$(find smb_description)/urdf/smb_rgb_camera.urdf.xacro"/>
     <!-- Defines lidar macro -->
     <xacro:include filename="$(find smb_description)/urdf/smb_lidar_mount.urdf.xacro"/>
@@ -161,7 +161,7 @@
         <xacro:IMU base_link="${base_link_name}" simulation="${simulation}"/>
         <!-- <xacro:GPS base_link="${base_link_name}" simulation="${simulation}"/> -->
-        <xacro:rgbcamera_cam id="" base_link="${base_link_name}" simulation="${simulation}">
+        <xacro:rgb_camera_cam id="" base_link="${base_link_name}" simulation="${simulation}">
             <origin xyz="0.29082 -0.04542 ${0.0955 + chassisHeight/2.0}" rpy="0 0 0" />
-        </xacro:rgbcamera_cam>
+        </xacro:rgb_camera_cam>
         <xacro:if value="${lidar}">
             <xacro:lidar_mount base_link="${base_link_name}"/>

File: smb_description/urdf/smb_rgb_camera.urdf.xacro (robot description, xacro)
@@ -4,13 +4,13 @@
 <robot name="smb" xmlns:xacro="http://www.ros.org/wiki/xacro">
   <!-- INCLUDE PLUGIN -->
-  <xacro:include filename="$(find smb_description)/urdf/sensor_plugins/smb_rgbcamera.gazebo.xacro"/>
-  <xacro:macro name="rgbcamera_cam" params="*origin id base_link simulation">
+  <xacro:include filename="$(find smb_description)/urdf/sensor_plugins/smb_rgb_camera.gazebo.xacro"/>
+  <xacro:macro name="rgb_camera_cam" params="*origin id base_link simulation">
     <!--                              Camera  Properties 				          	-->
-    <xacro:property name="rgbcamera_base_link"		value="${base_link}"/>
-    <xacro:property name="rgbcamera_origin_rpy"		value="0 0 0"/>
-    <xacro:property name="rgbcamera_origin_xyz"		value="0.29082 -0.04458 ${0.0955 + chassisHeight/2.0}"/>
-    <xacro:property name="rgbcamera_update_rate"		value="2"/>
-    <xacro:property name="rgbcamera_link"  			value="rgbcamera${id}_link"/>
-    <link name="${rgbcamera_link}">
+    <xacro:property name="rgb_camera_base_link"		value="${base_link}"/>
+    <xacro:property name="rgb_camera_origin_rpy"		value="0 0 0"/>
+    <xacro:property name="rgb_camera_origin_xyz"		value="0.29082 -0.04458 ${0.0955 + chassisHeight/2.0}"/>
+    <xacro:property name="rgb_camera_update_rate"		value="2"/>
+    <xacro:property name="rgb_camera_link"  			value="rgb_camera${id}_link"/>
+    <link name="${rgb_camera_link}">
       <inertial>
         <mass value="0.01" /> <!-- [kg] -->
@@ -31,24 +31,24 @@
         </material>
     </link>
-      <gazebo reference="${rgbcamera_link}">
+      <gazebo reference="${rgb_camera_link}">
         <material>Gazebo/Red</material>
       </gazebo>
-    <joint name="rgbcamera${id}_camera_joint" type="fixed">
-      <!-- <origin xyz="${rgbcamera_origin_xyz}" rpy="${rgbcamera_origin_rpy}"/> -->
+    <joint name="rgb_camera${id}_camera_joint" type="fixed">
+      <!-- <origin xyz="${rgb_camera_origin_xyz}" rpy="${rgb_camera_origin_rpy}"/> -->
       <xacro:insert_block name="origin"/>
-      <parent link="${rgbcamera_base_link}"/>
-      <child link="${rgbcamera_link}"/>
+      <parent link="${rgb_camera_base_link}"/>
+      <child link="${rgb_camera_link}"/>
     </joint>
-      <gazebo reference="rgbcamera${id}_camera_joint">
+      <gazebo reference="rgb_camera${id}_camera_joint">
         <disableFixedJointLumping>true</disableFixedJointLumping>
       </gazebo>
-    <link name="rgbcamera${id}_optical_link"/>
-    <joint name="rgbcamera${id}_camera_optical_joint" type="fixed">
+    <link name="rgb_camera${id}_optical_link"/>
+    <joint name="rgb_camera${id}_camera_optical_joint" type="fixed">
       <origin xyz="0.0066 0 0" rpy="-1.57 0 -1.57"/>
-      <parent link="${rgbcamera_link}"/>
-      <child link="rgbcamera${id}_optical_link"/>
+      <parent link="${rgb_camera_link}"/>
+      <child link="rgb_camera${id}_optical_link"/>
     </joint>
     <xacro:if value="${simulation}">
-        <xacro:rgbcamera_camera_plugin name="rgb_camera" link_name="${rgbcamera_link}" rate="${rgbcamera_update_rate}"/>
+        <xacro:rgb_camera_camera_plugin name="rgb_camera" link_name="${rgb_camera_link}" rate="${rgb_camera_update_rate}"/>
     </xacro:if>
   </xacro:macro>
